File: Catcar_Ringlight/led_group.kicad_sch (KiCad schematic)
At the start: 24 parts

Commit message: Change orange LED type
Other:
- note added: "White LEDs: WW-WNA30TS-U1(M1) Orange LEDs: OSY5CAS3C1A"
- note removed: "White LEDs: WW-WNA30TS-U1(M1) Orange LEDs: OSO5CAS3C1A"
Changed lines of the file:
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@@
   (title_block
     (title "LED Group")
-    (date "2023-07-18")
+    (date "2023-08-02")
     (rev "1.0")
     (company "xatLabs")
@@
     (stroke (width 0) (type default))
   )
-  (text "White LEDs: WW-WNA30TS-U1(M1)\nOrange LEDs: OSO5CAS3C1A"
+  (text "White LEDs: WW-WNA30TS-U1(M1)\nOrange LEDs: OSY5CAS3C1A"
     (at 124.46 107.95 0)
     (effects (font (size 1.27 1.27)) (justify left bottom))
